File: STM32_Controller_v3/Mcu_Stm32_sch.kicad_sch (KiCad schematic)
At the start: 43 parts, among them CN10 DS1021-1x5SF11-B, CN8 DS1021-1x4SF11-B, CN9 DS1021-1x6SF11-B, Q13 SMMBT5551LT1G, Q14 SMMBT5551LT1G, U3 STM32L151C8T6A

Commit message: production version
Parts:
- C19, C20, C21, C24, C26, C28: Assembly (none) -> SMT; Manufacturer (none) -> YAGEO; Part.Number (none) -> CC0805KRX7R9BB104
- DS1: Assembly (none) -> PTH; Part.Number (none) -> MGD1602A-NSW-BBS-01
- LD13: Assembly (none) -> SMT; Manufacturer (none) -> NATIONSTAR; Part.Number (none) -> NCD0805R1
- Q13, Q14: Assembly (none) -> SMT; Manufacturer (none) -> JSCJ; Part.Number (none) -> MMBT5551
- R35: Assembly (none) -> SMT; Manufacturer (none) -> UNI-ROYAL; Part.Number (none) -> 0805W8F0000T5E
- R49, R60, R63, R74: Assembly (none) -> SMT; Manufacturer (none) -> UNI-ROYAL; Part.Number (none) -> 0805W8F1001T5E
- R50, R51, R53, R55, R56, R57, R58, R61, R62, R64, R67, R68, R72, R75: Assembly (none) -> SMT; Manufacturer (none) -> UNI-ROYAL; Part.Number (none) -> 0805W8F1002T5E
- R59, R65, R66, R69, R70, R73, R86, R87: Assembly (none) -> SMT; Manufacturer (none) -> UNI-ROYAL; Part.Number (none) -> 0805W8F1200T5E
- R85: Assembly (none) -> SMT; Manufacturer (none) -> UNI-ROYAL; Part.Number (none) -> 0805W8F100JT5E
- U3: Assembly (none) -> SMT; Manufacturer (none) -> ST; Part.Number (none) -> STM32L151C8T6
Connections:
- net LCD_BKL: now also U3.2 (PC13); no longer U3.38 (PA15)
- net LCD_D5: now also U3.43 (PB7); no longer U3.41 (PB5)
- net LCD_D6: now also U3.45 (PB8); no longer U3.40 (PB4)
- net LCD_D7: now also U3.46 (PB9); no longer U3.39 (PB3)
- net LCD_E: now also U3.41 (PB5); no longer U3.43 (PB7)
- net LCD_RS: now also U3.39 (PB3); no longer U3.46 (PB9)
- net LCD_RW: now also U3.40 (PB4); no longer U3.45 (PB8)
