File: STM32_Controller_v3/Power_Supply_sch.kicad_sch (KiCad schematic)
At the start: 43 parts, among them CN3 WJ15EDGVC-3.5-02P-14-00A, U1 TPS5430DDA, U2 MIC5504-3.3YM5, U5 TPS2553DBVR, U7 TPS2553DBVR

Commit message: production version
Parts:
- removed CN3: WJ15EDGVC-3.5-02P-14-00A, Library:PhoenixContact_MCV_1,5_2-G-3.5_1x02_P3.50mm_Vertical, symbol Library:CN_Header_3.5mm_2W_180_300V
- removed CNP3: WJ15EDGK-3.5-02P-14-00A, symbol Library:CN_Plug_3.5mm_2W_180_300V
- added CN3: WJ15EDGVC-3.81-02P-14-00A, Library:PhoenixContact_MCV_1,5_2-G-3.81_1x02_P3.81mm_Vertical, symbol Library:CN_Header_3.81mm_2W_180_300V
- added CNP3: WJ15EDGK-3.81-02P-14-00A, symbol Library:CN_Plug_3.81mm_2W_180_300V
- added H1, H2, H3, H4: MountingHole, Library:MountingHole_4.3mm_M4_Pad_Via, symbol Library:MountingHole
- C10, C9: footprint db_capacitors:C_1206 -> Library:C_1206; Assembly (none) -> SMT; Manufacturer (none) -> FH; Part.Number (none) -> 1206B475K500NT
- C11: footprint db_capacitors:C_0805 -> Library:C_0805; Assembly (none) -> SMT; Manufacturer (none) -> Samsung Electro-Mechanics; Part.Number (none) -> CL21B103KBANNNC
- C13, C14: Assembly (none) -> SMT; Manufacturer (none) -> Lelon; Part.Number (none) -> VEJ101M1HTR-0810L
- C16, C18, C23, C34, C35, C38, C41: Assembly (none) -> SMT; Manufacturer (none) -> YAGEO; Part.Number (none) -> CC0805KRX7R9BB104
- C17, C22, C31: Assembly (none) -> SMT; Manufacturer (none) -> Samsung Electro-Mechanics; Part.Number (none) -> CL21B105KBFNNNE
- C33, C40: Assembly (none) -> SMT; Manufacturer (none) -> Kyocera AVX; Part.Number (none) -> TPSB476K010R0350
- D10, D8: Assembly (none) -> SMT; Manufacturer (none) -> MDD(Microdiode Semiconductor); Part.Number (none) -> SS14
- D5: Assembly (none) -> SMT; Manufacturer (none) -> RUILON; Part.Number (none) -> SMAJ26A
- FD1, FD2, FD3: now not fitted
- L1, L2: Assembly (none) -> SMT; Manufacturer (none) -> muRata; Part.Number (none) -> BLM18KG601SN1D
- L4: value FNR6045S220MT -> 22uF; Assembly (none) -> SMT; Manufacturer (none) -> cjiang; Part.Number (none) -> FNR6045S220MT
- R36: Assembly (none) -> SMT; Manufacturer (none) -> UNI-ROYAL; Part.Number (none) -> 0805W8F3241T5E
- R52, R82: Assembly (none) -> SMT; Manufacturer (none) -> UNI-ROYAL; Part.Number (none) -> 0805W8F0000T5E
- R71: Assembly (none) -> SMT; Manufacturer (none) -> UNI-ROYAL; Part.Number (none) -> 0805W8F1002T5E
- R79, R80, R83, R84: Assembly (none) -> SMT; Manufacturer (none) -> YAGEO; Part.Number (none) -> RC0805FR-07100KL
- U1: Assembly (none) -> SMT; Manufacturer (none) -> TI; Part.Number (none) -> TPS5430DDAR
- U2: Assembly (none) -> SMT; Manufacturer (none) -> MICROCHIP; Part.Number (none) -> MIC5504-3.3YM5-TR
- U5, U7: Assembly (none) -> SMT; Manufacturer (none) -> TI; Part.Number (none) -> TPS2553DBVR
Connections:
- net +3.3V: no longer R83.2
- net +3.3V_P: now also R83.2
- net +V_IN: now also CN3.2 (Pin_2)
- net GND: now also CN3.1 (Pin_1)
- net TPS_FB: now reaches R36.1, R71.2, U1.4 (VSENSE)
- net TPS_VIN: now reaches C10.1, C16.1, C9.1, L1.2, U1.7 (VIN)
- net TPS_PH: now reaches C11.2, D10.1 (K), L4.1, U1.8 (PH)
- net TPS_BOOT: now reaches C11.1, U1.1 (BOOT)
