File: STM32_Controller_v3/Power_Supply_sch.kicad_sch (KiCad schematic)
At the start: 47 parts, among them CN3 WJ15EDGVC-3.81-02P-14-00A, U1 TPS5430DDA, U2 MIC5504-3.3YM5, U5 TPS2553DBVR, U7 TPS2553DBVR

Commit message: update dimension information
Other:
- note added: "VIN: 9 to 24VDC"
Changed lines of the file:
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@@
 		(comment 2 "29/08/2025")
+	)
+	(text "VIN: 9 to 24VDC"
+		(exclude_from_sim no)
+		(at 46.228 17.272 0)
+		(effects
+			(font
+				(size 1.27 1.27)
+			)
+		)
 	)
 	(junction
