File: STM32_Controller_v3/Power_Supply_sch.kicad_sch (KiCad schematic)
At the start: 47 parts, among them CN3 WJ15EDGVC-3.81-02P-14-00A, U1 TPS5430DDA, U2 MIC5504-3.3YM5, U5 TPS2553DBVR, U7 TPS2553DBVR

Commit message: res 4k7 in digital inputs and outputs leds
Parts:
- R36: value 1K -> 3K24
Changed lines of the file:
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@@
 			)
 		)
-		(property "Value" "1K"
+		(property "Value" "3K24"
 			(at 241.3 63.4999 0)
 			(show_name no)
